File: rpi-hat/rpi-hat.sch (KiCad schematic (older format))
At the start: 31 parts, among them J1 Raspberry_Pi_2_3, J2 UEXT_Slave, J3 RJ45_Shielded, J4 DB9 Male CAN, J5 Screw_Terminal_01x02, U1 CAT24C128, U2 MCP2517FD-xSL, U3 SN65HVD235, Y1 20MHz

Commit message: Fix problems with project-specific library
Use 1206/3216Metric footprints for all capacitors and resistors.
Fix QR code to be negative and to point to the proper address.
Parts:
- C2, C3, C4, C5: footprint Capacitor_SMD:C_0603_1608Metric_Pad1.05x0.95mm_HandSolder -> Capacitor_SMD:C_1206_3216Metric_Pad1.42x1.75mm_HandSolder
- R4, R5, R6: footprint Resistor_SMD:R_0603_1608Metric_Pad1.05x0.95mm_HandSolder -> Resistor_SMD:R_1206_3216Metric_Pad1.42x1.75mm_HandSolder
Changed lines of the file:
@@
 F 0 "C5" V 7700 2600 50  0000 C CNN
 F 1 "100nF" V 7950 2700 50  0000 C CNN
-F 2 "Capacitor_SMD:C_0603_1608Metric_Pad1.05x0.95mm_HandSolder" H 7850 2600 50  0001 C CNN
+F 2 "Capacitor_SMD:C_1206_3216Metric_Pad1.42x1.75mm_HandSolder" H 7850 2600 50  0001 C CNN
 F 3 "~" H 7850 2600 50  0001 C CNN
 F 4 "EMK107B7104KAHT" V 7850 2600 50  0001 C CNN "Mfg"
@@
 F 0 "C4" V 6400 2600 50  0000 C CNN
 F 1 "100nF" V 6650 2700 50  0000 C CNN
-F 2 "Capacitor_SMD:C_0603_1608Metric_Pad1.05x0.95mm_HandSolder" H 6550 2600 50  0001 C CNN
+F 2 "Capacitor_SMD:C_1206_3216Metric_Pad1.42x1.75mm_HandSolder" H 6550 2600 50  0001 C CNN
 F 3 "~" H 6550 2600 50  0001 C CNN
 F 4 "EMK107B7104KAHT" V 6550 2600 50  0001 C CNN "Mfg"
@@
 F 0 "C2" H 5315 3846 50  0000 L CNN
 F 1 "22pF" H 5315 3755 50  0000 L CNN
-F 2 "Capacitor_SMD:C_0603_1608Metric_Pad1.05x0.95mm_HandSolder" H 5238 3650 50  0001 C CNN
+F 2 "Capacitor_SMD:C_1206_3216Metric_Pad1.42x1.75mm_HandSolder" H 5238 3650 50  0001 C CNN
 F 3 "~" H 5200 3800 50  0001 C CNN
 F 4 "06035C220JAT2A" H 5200 3800 50  0001 C CNN "Mfg"
@@
 F 0 "C3" H 5815 3846 50  0000 L CNN
 F 1 "22pF" H 5815 3755 50  0000 L CNN
-F 2 "Capacitor_SMD:C_0603_1608Metric_Pad1.05x0.95mm_HandSolder" H 5738 3650 50  0001 C CNN
+F 2 "Capacitor_SMD:C_1206_3216Metric_Pad1.42x1.75mm_HandSolder" H 5738 3650 50  0001 C CNN
 F 3 "~" H 5700 3800 50  0001 C CNN
 F 4 "06035C220JAT2A" H 5700 3800 50  0001 C CNN "Mfg"
@@
 F 0 "R4" H 7570 3446 50  0000 L CNN
 F 1 "100k" H 7570 3355 50  0000 L CNN
-F 2 "Resistor_SMD:R_0603_1608Metric_Pad1.05x0.95mm_HandSolder" V 7430 3400 50  0001 C CNN
+F 2 "Resistor_SMD:R_1206_3216Metric_Pad1.42x1.75mm_HandSolder" V 7430 3400 50  0001 C CNN
 F 3 "~" H 7500 3400 50  0001 C CNN
 F 4 "CRCW0603100KFKEAC" H 7500 3400 50  0001 C CNN "Mfg"
@@
 F 0 "R5" H 6420 5646 50  0000 L CNN
 F 1 "120" H 6420 5555 50  0000 L CNN
-F 2 "Resistor_SMD:R_0603_1608Metric_Pad1.05x0.95mm_HandSolder" V 6280 5600 50  0001 C CNN
+F 2 "Resistor_SMD:R_1206_3216Metric_Pad1.42x1.75mm_HandSolder" V 6280 5600 50  0001 C CNN
 F 3 "~" H 6350 5600 50  0001 C CNN
 F 4 "CRCW0603120RFKEAC" H 6350 5600 50  0001 C CNN "Mfg"
@@
 F 0 "R6" H 6720 5546 50  0000 L CNN
 F 1 "120" H 6720 5455 50  0000 L CNN
-F 2 "Resistor_SMD:R_0603_1608Metric_Pad1.05x0.95mm_HandSolder" V 6580 5500 50  0001 C CNN
+F 2 "Resistor_SMD:R_1206_3216Metric_Pad1.42x1.75mm_HandSolder" V 6580 5500 50  0001 C CNN
 F 3 "~" H 6650 5500 50  0001 C CNN
 F 4 "CRCW0603120RFKEAC" H 6650 5500 50  0001 C CNN "Mfg"
